File: Hardware/Kicad files/USB_DAC/USB_DAC.kicad_sch (KiCad schematic)
At the start: 0 parts

Commit message: Updated PCB and schematics
Other:
- company: (none) -> Linus Fridlund
Changed lines of the file:
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@@
 	(generator_version "9.0")
 	(paper "A4")
+	(title_block
+		(rev "1.0")
+		(company "Linus Fridlund")
+	)
 	(sheet
 		(at 143.51 22.86)
