File: Hardware/Kicad files/USB_DAC/DAC_DAC.kicad_sch (KiCad schematic)
At the start: 42 parts, among them IC1 ES9039Q2M, IC2 LT3094EDD_PBF, U4 OPA1612AxD, U5 OPA1612AxD, U6 LT3042IMSE_PBF, U7 TPS7A2033PDBVR, Y3 NSC5083D

Commit message: Updated PCB and schematics
Connections:
- net DC_IN: now reaches C16.1, C17.1, C33.1, PS1.2 (+VIN_(VCC))
Other:
- note added: "Analog power supply"
- note added: "As shown in DAC datasheet"
- note added: "CH1 Output stage"
- note added: "CH2 Output stage"
- note added: "DAC Chip"
- note added: "ES9039Q2M"
- note added: "TODO: - LDO for +-9VA - LDO for OSC + DAC chip"
- note removed: "CH1 OUT"
- note removed: "CH2 OUT"
- note removed: "DAC CHIP"
- note removed: "PWR SUPPLY"
- note removed: "TODO: - LDO for +-9VA - LDO for OSC + DAC chip - Pullups for I2C"
- company: (none) -> Linus Fridlund
- title: (none) -> DAC Sheet
- moved on the sheet: C14, C15, C16, C17, C18, C32, C33, C37, C38, C39, C40, C41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

Commit message: Updated PCB and schematics
Parts:
- added C53, C54, C55, C56, C57, C58: 4u7, Capacitor_SMD:C_1206_3216Metric, symbol Device:C_Small
- added C59, C60: 100n, Capacitor_SMD:C_0603_1608Metric, symbol Device:C_Small
- added R29, R30: 90k 1%, Resistor_SMD:R_0603_1608Metric, symbol Device:R
Connections:
- net +12VA is gone; now on net +12V: C14.1, C18.1, PS1.6 (+VOUT)
- net -12VA is gone; now on net -12V: C15.2, C32.2, PS1.8 (-VOUT)
- net +3.3VA: now also U7.5 (OUT), C60.1
- net +9VA: now also U6.10 (OUT), U6.9 (OUTS), U7.1 (IN), U7.3 (EN), C54.1, C59.1
- net -9VA: now also IC2.10 (OUTS), IC2.11 (OUT_1), IC2.12 (OUT_2), C58.1
- net GND: now also C14.2, C15.1, C18.2, C32.1, C37.1, C38.2, C39.1, C40.1, C41.2, IC1.11 (GND_1), IC1.17 (RT1), IC1.19 (SS/ADDR1/HW2), IC1.20 (MISO/ADDR0/MUTE_CTRL), IC1.29 (MODE), IC1.30 (GND_2), IC1.33 (GND_3), IC2.6 (ILIM), IC2.9 (GND), PS1.7 (COMMON), U4.3 (+), U5.3 (+), U6.5 (ILIM), U7.2 (GND), Y3.2 (GND), C53.2, C54.2, C55.2, C56.2, C57.2, C58.2, C59.2, C60.2, R29.1, R30.1
- net GNDA: no longer C14.2, C15.1, C18.2, C32.1, C37.1, C38.2, C39.1, C40.1, C41.2, IC1.11 (GND_1), IC1.17 (RT1), IC1.19 (SS/ADDR1/HW2), IC1.20 (MISO/ADDR0/MUTE_CTRL), IC1.29 (MODE), IC1.30 (GND_2), IC1.33 (GND_3), PS1.7 (COMMON), U4.3 (+), U5.3 (+), Y3.2 (GND)
- net +12V: now reaches U6.1 (IN), U6.2 (IN)
- net +12V: now also U6.3 (EN/UV), U6.6 (PGFB), C55.1
- net at U6.7 (SET): now also C53.1, R29.2
- net -12V: now reaches IC2.1 (IN_1)
- net -12V: now also IC2.2 (IN_2), IC2.3 (EN/UV), IC2.5 (PGFB), C57.1
- net at IC2.8 (SET): now also C56.1, R30.2
Other:
- note removed: "TODO: - LDO for +-9VA - LDO for OSC + DAC chip"
- moved on the sheet: C14, C15, C16, C17, C18, C32, C33, C37, C38, C39, C40, C41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
